File: eagle/PandionVTOL/transition_control_arduino.brd (EAGLE design)
At the start: 62.2 x 64.4 mm, 7 parts, among them IC1 L293D, M1 JST-XH-02-PIN-ROUND-PAD, M2 JST-XH-02-PIN-ROUND-PAD

Commit message: Working on transition
Connections:
- new net 3V3: ARDUINO_NANO1.2, COM1.2, COM2.2
- new net VCC: ARDUINO_NANO1.12, IC1.16
- net 5V: no longer ARDUINO_NANO1.12, COM1.2, COM2.2, IC1.16
- net D2: no longer IC1.9
- net D5: now also IC1.9
Routing:
- net 3V3: track 0.00 -> 112.6 mm
- net 5V: track 126.2 -> 39.3 mm
- net VCC: track 0.00 -> 64.8 mm
- net D5: track 0.00 -> 47.2 mm
- net D2: track 25.9 -> 0.00 mm
Other:
- board size 62.2 x 64.4 mm -> 62.2 x 67 mm
Changed lines of the file:
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@@
 <?xml version="1.0" encoding="utf-8"?>
 <!DOCTYPE eagle SYSTEM "eagle.dtd">
-<eagle version="9.5.2">
+<eagle version="9.2.2">
 <drawing>
 <settings>
@@
 <plain>
 <wire x1="97.79" y1="35.56" x2="160" y2="35.56" width="0" layer="20"/>
-<wire x1="160" y1="35.56" x2="160" y2="100" width="0" layer="20"/>
-<wire x1="160" y1="100" x2="97.79" y2="100" width="0" layer="20"/>
-<wire x1="97.79" y1="100" x2="97.79" y2="35.56" width="0" layer="20"/>
+<wire x1="160" y1="35.56" x2="160" y2="102.54" width="0" layer="20"/>
+<wire x1="160" y1="102.54" x2="97.79" y2="102.54" width="0" layer="20"/>
+<wire x1="97.79" y1="102.54" x2="97.79" y2="35.56" width="0" layer="20"/>
 </plain>
 <attributes>
@@
 <wire x1="104.14" y1="49.57" x2="104.14" y2="58.42" width="0.8128" layer="1"/>
 <wire x1="104.14" y1="58.42" x2="106.68" y2="60.96" width="0.8128" layer="1"/>
-<wire x1="115.99555625" y1="41.1607" x2="116.74485625" y2="41.91" width="0.8128" layer="1"/>
 <wire x1="110.53" y1="43.18" x2="112.5493" y2="41.1607" width="0.8128" layer="1"/>
-<wire x1="112.5493" y1="41.1607" x2="115.99555625" y2="41.1607" width="0.8128" layer="1"/>
 <wire x1="134.62" y1="82.55" x2="129.54" y2="77.47" width="0.8128" layer="16"/>
 <wire x1="129.54" y1="77.47" x2="120.65" y2="77.47" width="0.8128" layer="16"/>
@@
 <contactref element="COM1" pad="1"/>
 <contactref element="COM2" pad="1"/>
-<wire x1="116.74485625" y1="41.91" x2="140.97" y2="41.91" width="0.8128" layer="1"/>
+<wire x1="140.2207" y1="41.1607" x2="140.97" y2="41.91" width="0.8128" layer="1"/>
+<wire x1="140.2207" y1="41.1607" x2="112.5493" y2="41.1607" width="0.8128" layer="1"/>
 <wire x1="140.97" y1="41.91" x2="153.67" y2="41.91" width="0.8128" layer="1"/>
 <wire x1="106.68" y1="60.96" x2="121.92" y2="66.04" width="0" layer="19" extent="1-1"/>
@@
 <signal name="D5" class="1">
 <contactref element="ARDUINO_NANO1" pad="23"/>
+<contactref element="IC1" pad="9"/>
+<wire x1="144.1196" y1="88.1350125" x2="143.51" y2="88.7446125" width="0.8128" layer="16"/>
+<wire x1="143.51" y1="88.7446125" x2="143.51" y2="88.9" width="0.8128" layer="16"/>
+<wire x1="144.1196" y1="74.2696" x2="144.1196" y2="88.1350125" width="0.8128" layer="16"/>
+<wire x1="142.24" y1="72.39" x2="144.1196" y2="74.2696" width="0.8128" layer="16"/>
+<wire x1="130.81" y1="76.2" x2="121.92" y2="76.2" width="0.8128" layer="16"/>
+<wire x1="136.4996" y1="79.5049875" x2="135.7854125" y2="78.7908" width="0.8128" layer="16"/>
+<wire x1="143.51" y1="88.9" x2="143.4592" y2="88.8492" width="0.8128" layer="16"/>
+<wire x1="133.4008" y1="78.7908" x2="130.81" y2="76.2" width="0.8128" layer="16"/>
+<wire x1="143.4592" y1="88.8492" x2="141.0745875" y2="88.8492" width="0.8128" layer="16"/>
+<wire x1="135.7854125" y1="78.7908" x2="133.4008" y2="78.7908" width="0.8128" layer="16"/>
+<wire x1="141.0745875" y1="88.8492" x2="136.4996" y2="84.2742125" width="0.8128" layer="16"/>
+<wire x1="136.4996" y1="84.2742125" x2="136.4996" y2="79.5049875" width="0.8128" layer="16"/>
 </signal>
 <signal name="D6" class="1">
@@
 </signal>
 <signal name="5V" class="1">
-<contactref element="IC1" pad="16"/>
-<contactref element="IC1" pad="8"/>
-<contactref element="ARDUINO_NANO1" pad="12"/>
 <contactref element="X1" pad="1"/>
-<wire x1="115.53" y1="43.18" x2="116.8" y2="44.45" width="0.8128" layer="1"/>
-<wire x1="115.53" y1="43.18" x2="109.22" y2="49.49" width="0.8128" layer="1"/>
-<wire x1="109.22" y1="49.49" x2="109.22" y2="63.5" width="0.8128" layer="1"/>
-<wire x1="109.22" y1="63.5" x2="106.68" y2="66.04" width="0.8128" layer="1"/>
-<wire x1="134.62" y1="72.39" x2="137.16" y2="74.93" width="0.8128" layer="16"/>
-<wire x1="137.16" y1="74.93" x2="137.16" y2="86.36" width="0.8128" layer="16"/>
-<wire x1="137.16" y1="86.36" x2="140.97" y2="90.17" width="0.8128" layer="16"/>
-<wire x1="140.97" y1="90.17" x2="142.24" y2="90.17" width="0.8128" layer="16"/>
-<contactref element="COM1" pad="2"/>
-<contactref element="COM2" pad="2"/>
-<wire x1="116.8" y1="44.45" x2="140.97" y2="44.45" width="0.8128" layer="1"/>
-<wire x1="140.97" y1="44.45" x2="153.67" y2="44.45" width="0.8128" layer="1"/>
-<wire x1="134.62" y1="72.39" x2="124.46" y2="62.23" width="0.8128" layer="1"/>
-<wire x1="124.46" y1="62.23" x2="120.65" y2="62.23" width="0.8128" layer="1"/>
+<wire x1="120.65" y1="62.23" x2="124.46" y2="62.23" width="0.8128" layer="1"/>
 <wire x1="120.65" y1="62.23" x2="115.53" y2="57.11" width="0.8128" layer="1"/>
 <wire x1="115.53" y1="57.11" x2="115.53" y2="43.18" width="0.8128" layer="1"/>
+<contactref element="IC1" pad="8"/>
+<wire x1="124.46" y1="62.23" x2="134.62" y2="72.39" width="0.8128" layer="1"/>
 </signal>
 <signal name="D2" class="1">
 <contactref element="ARDUINO_NANO1" pad="20"/>
-<wire x1="123.19" y1="67.31" x2="121.92" y2="68.58" width="0.8128" layer="16"/>
-<contactref element="IC1" pad="9"/>
-<wire x1="142.24" y1="72.39" x2="142.24" y2="67.31" width="0.8128" layer="16"/>
-<wire x1="142.24" y1="67.31" x2="123.19" y2="67.31" width="0.8128" layer="16"/>
 </signal>
 <signal name="M2A" class="1">
@@
 <signal name="N$1" class="1">
 <polygon width="0.8128" layer="16">
-<vertex x="97.79" y="100.33"/>
-<vertex x="160.02" y="100.33"/>
+<vertex x="97.79" y="102.87"/>
+<vertex x="160.02" y="102.87"/>
 <vertex x="160.02" y="35.56"/>
 <vertex x="97.79" y="35.56"/>
 </polygon>
 </signal>
+<signal name="VCC" class="1">
+<contactref element="ARDUINO_NANO1" pad="12"/>
+<contactref element="IC1" pad="16"/>
+<wire x1="142.24" y1="90.17" x2="133.35" y2="99.06" width="0.8128" layer="1"/>
+<wire x1="133.35" y1="99.06" x2="119.38" y2="99.06" width="0.8128" layer="1"/>
+<wire x1="119.38" y1="99.06" x2="119.38" y2="78.74" width="0.8128" layer="1"/>
+<wire x1="119.38" y1="78.74" x2="106.68" y2="66.04" width="0.8128" layer="1"/>
+</signal>
+<signal name="3V3" class="1">
+<contactref element="ARDUINO_NANO1" pad="2"/>
+<contactref element="COM1" pad="2"/>
+<contactref element="COM2" pad="2"/>
+<wire x1="140.97" y1="44.45" x2="153.67" y2="44.45" width="0.8128" layer="1"/>
+<wire x1="153.67" y1="44.45" x2="157.48" y2="48.26" width="0.8128" layer="1"/>
+<wire x1="157.48" y1="48.26" x2="157.48" y2="78.74" width="0.8128" layer="1"/>
+<wire x1="135.1024" y1="101.1176" x2="123.19" y2="101.1176" width="0.8128" layer="1"/>
+<wire x1="123.19" y1="101.1176" x2="123.13121875" y2="101.1176" width="0.8128" layer="1"/>
+<wire x1="157.48" y1="78.74" x2="135.1024" y2="101.1176" width="0.8128" layer="1"/>
+<wire x1="123.13121875" y1="101.1176" x2="116.3576" y2="101.1176" width="0.8128" layer="1"/>
+<wire x1="116.3576" y1="101.1176" x2="106.68" y2="91.44" width="0.8128" layer="1"/>
+</signal>
 </signals>
