File: eagle/PandionVTOL/transition_control_arduino.sch (EAGLE design)
At the start: 7 parts, among them IC1 L293D, M1 JST-XH-02-PIN-ROUND-PAD, M2 JST-XH-02-PIN-ROUND-PAD

Commit message: Working on transition
Connections:
- new net 3V3: ARDUINO_NANO1.3V3, COM1-2.S, COM2-2.S
- new net VCC: ARDUINO_NANO1.5V, IC1.VCC1
- net 5V: no longer ARDUINO_NANO1.5V, COM1-2.S, COM2-2.S, IC1.VCC1
- net D2: no longer IC1.3-4EN
- net D5: now also IC1.3-4EN
Other:
- note added: "PWM"
