File: eagle/PandionVTOL/transition_control_esp32.brd (EAGLE design)
At the start: 160 x 100 mm, 8 parts, among them U1 ESP32-DEVKITC-32D

Commit message: esp32 board update
Parts:
- moved SV1 74.2 mm to (24.1, 68.6), turned to 270 degrees
Routing:
- net APROP: track 38.2 -> 75.1 mm
- net 5V: track 102.7 -> 113.0 mm
- net GND: track 181.4 -> 191.7 mm
- net ELEV: track 76.3 -> 84.0 mm
- net RUD: track 69.6 -> 77.3 mm
Changed lines of the file:
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@@
 <attribute name="VALUE" x="28.829" y="81.28" size="1.27" layer="27" ratio="10" rot="R270"/>
 </element>
-<element name="SV1" library="con-lstb" library_urn="urn:adsk.eagle:library:162" package="MA05-1" package3d_urn="urn:adsk.eagle:package:8332/1" value="" x="7.62" y="-3.81" smashed="yes">
-<attribute name="MF" value="" x="7.62" y="-3.81" size="1.778" layer="27" display="off"/>
-<attribute name="MPN" value="" x="7.62" y="-3.81" size="1.778" layer="27" display="off"/>
-<attribute name="NAME" x="1.27" y="-2.159" size="1.27" layer="25" ratio="10"/>
-<attribute name="OC_FARNELL" value="unknown" x="7.62" y="-3.81" size="1.778" layer="27" display="off"/>
-<attribute name="OC_NEWARK" value="unknown" x="7.62" y="-3.81" size="1.778" layer="27" display="off"/>
-<attribute name="POPULARITY" value="29" x="7.62" y="-3.81" size="1.778" layer="27" display="off"/>
-<attribute name="VALUE" x="5.08" y="-6.731" size="1.27" layer="27" ratio="10"/>
+<element name="SV1" library="con-lstb" library_urn="urn:adsk.eagle:library:162" package="MA05-1" package3d_urn="urn:adsk.eagle:package:8332/1" value="" x="24.13" y="68.58" smashed="yes" rot="R270">
+<attribute name="MF" value="" x="24.13" y="68.58" size="1.778" layer="27" rot="R270" display="off"/>
+<attribute name="MPN" value="" x="24.13" y="68.58" size="1.778" layer="27" rot="R270" display="off"/>
+<attribute name="NAME" x="25.781" y="74.93" size="1.27" layer="25" ratio="10" rot="R270"/>
+<attribute name="OC_FARNELL" value="unknown" x="24.13" y="68.58" size="1.778" layer="27" rot="R270" display="off"/>
+<attribute name="OC_NEWARK" value="unknown" x="24.13" y="68.58" size="1.778" layer="27" rot="R270" display="off"/>
+<attribute name="POPULARITY" value="29" x="24.13" y="68.58" size="1.778" layer="27" rot="R270" display="off"/>
+<attribute name="VALUE" x="21.209" y="71.12" size="1.27" layer="27" ratio="10" rot="R270"/>
 </element>
 </elements>
@@
 <wire x1="95.25" y1="79.248" x2="95.25" y2="79.3" width="0.4064" layer="16"/>
 <contactref element="SV1" pad="2"/>
-<wire x1="5.08" y1="-3.81" x2="31.75" y2="77.47" width="0" layer="19" extent="1-1"/>
+<wire x1="25.4508" y1="71.1708" x2="24.1554" y2="71.1708" width="0.4064" layer="16"/>
+<wire x1="31.75" y1="77.47" x2="25.4508" y2="71.1708" width="0.4064" layer="16"/>
+<wire x1="24.1554" y1="71.1708" x2="24.13" y2="71.12" width="0.4064" layer="16"/>
 </signal>
 <signal name="GND" class="1">
@@
 <wire x1="95.25" y1="66.675" x2="95.25" y2="66.6" width="0.4064" layer="16"/>
 <contactref element="SV1" pad="1"/>
-<wire x1="2.54" y1="-3.81" x2="85.09" y2="19.05" width="0" layer="19" extent="1-1"/>
+<wire x1="25.4508" y1="73.6854" x2="24.1554" y2="73.6854" width="0.4064" layer="1"/>
+<wire x1="31.623" y1="79.8576" x2="25.4508" y2="73.6854" width="0.4064" layer="1"/>
+<wire x1="24.1554" y1="73.6854" x2="24.13" y2="73.66" width="0.4064" layer="1"/>
+<wire x1="31.623" y1="79.8576" x2="31.75" y2="80.01" width="0.4064" layer="1"/>
 </signal>
 <signal name="VCC" class="1">
@@
 <wire x1="95.25" y1="48.8442" x2="95.25" y2="48.82" width="0.4064" layer="16"/>
 <contactref element="SV1" pad="5"/>
-<wire x1="12.7" y1="-3.81" x2="31.7754" y2="63.4746" width="0" layer="19" extent="16-16"/>
+<wire x1="31.623" y1="63.5508" x2="24.1554" y2="63.5508" width="0.4064" layer="16"/>
+<wire x1="24.1554" y1="63.5508" x2="24.13" y2="63.5" width="0.4064" layer="16"/>
+<wire x1="31.623" y1="63.5508" x2="31.7754" y2="63.4746" width="0.4064" layer="16"/>
 </signal>
 <signal name="RUD" class="1">
@@
 <wire x1="95.25" y1="51.435" x2="95.25" y2="51.36" width="0.4064" layer="1"/>
 <contactref element="SV1" pad="4"/>
-<wire x1="10.16" y1="-3.81" x2="31.7754" y2="65.9892" width="0" layer="19" extent="1-1"/>
+<wire x1="31.623" y1="66.0654" x2="24.1554" y2="66.0654" width="0.4064" layer="1"/>
+<wire x1="24.1554" y1="66.0654" x2="24.13" y2="66.04" width="0.4064" layer="1"/>
+<wire x1="31.623" y1="66.0654" x2="31.7754" y2="65.9892" width="0.4064" layer="1"/>
 </signal>
 <signal name="APROP" class="1">
@@
 <wire x1="95.25" y1="59.055" x2="95.25" y2="58.98" width="0.4064" layer="16"/>
 <contactref element="SV1" pad="3"/>
-<wire x1="7.62" y1="-3.81" x2="61.1124" y2="68.58" width="0" layer="19" extent="16-16"/>
+<wire x1="61.1124" y1="68.58" x2="24.13" y2="68.58" width="0.4064" layer="16"/>
 </signal>
 </signals>
